File: MCU.kicad_sch (KiCad schematic)
At the start: 9 parts, among them J301 Conn_ARM_JTAG_SWD_10, U301 STM32F072RBTx

Commit message: Rename LCSC Field
Parts:
- C301, C302, C303, C304: LCSC Part C307331 -> (none); LCSC# (none) -> C307331
- C305: LCSC Part C16780 -> (none); LCSC# (none) -> C16780
- R301: LCSC Part C25804 -> (none); LCSC# (none) -> C25804
Changed lines of the file:
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@@
       (effects (font (size 1.27 1.27)) hide)
     )
-    (property "LCSC Part" "C25804" (id 4) (at 34.29 45.72 0)
+    (property "LCSC#" "C25804" (id 4) (at 34.29 45.72 0)
       (effects (font (size 1.27 1.27)) hide)
     )
@@
       (effects (font (size 1.27 1.27)) hide)
     )
-    (property "LCSC Part" "C16780" (id 4) (at 160.02 26.67 0)
+    (property "LCSC#" "C16780" (id 4) (at 160.02 26.67 0)
       (effects (font (size 1.27 1.27)) hide)
     )
@@
       (effects (font (size 1.27 1.27)) hide)
     )
-    (property "LCSC Part" "C307331" (id 4) (at 149.86 26.67 0)
+    (property "LCSC#" "C307331" (id 4) (at 149.86 26.67 0)
       (effects (font (size 1.27 1.27)) hide)
     )
@@
       (effects (font (size 1.27 1.27)) hide)
     )
-    (property "LCSC Part" "C307331" (id 4) (at 119.38 26.67 0)
+    (property "LCSC#" "C307331" (id 4) (at 119.38 26.67 0)
       (effects (font (size 1.27 1.27)) hide)
     )
@@
       (effects (font (size 1.27 1.27)) hide)
     )
-    (property "LCSC Part" "C307331" (id 4) (at 139.7 26.67 0)
+    (property "LCSC#" "C307331" (id 4) (at 139.7 26.67 0)
       (effects (font (size 1.27 1.27)) hide)
     )
@@
       (effects (font (size 1.27 1.27)) hide)
     )
-    (property "LCSC Part" "C307331" (id 4) (at 129.54 26.67 0)
+    (property "LCSC#" "C307331" (id 4) (at 129.54 26.67 0)
       (effects (font (size 1.27 1.27)) hide)
     )
